File: Gamble Boy.kicad_sch (KiCad schematic)
At the start: 3 parts, among them J1 Raspberry Pi Zero 2W, J2 128x160 SPI Display, SW1 Slider

Commit message: I FORGOT TO COMMIT FUCK FUCK FUCK
Parts:
- removed SW1: Slider, symbol Switch:SW_Slide_DPDT
- added SW1: SW_Push, symbol Switch:SW_Push
Connections:
- net GND: now also SW1.2
- net SliderVCC renamed BigButton
- net BigButton: now also SW1.1
